File: module_SIM800C.sch (KiCad schematic (older format))
At the start: 21 parts, among them J6 LEMO2, J7 SIM_Card, U5 SIM800C

Commit message: Add button to pin PWRKEY in SIM800C for handle power on SIM800C
Parts:
- removed R15: 10k, footprint:R_0603, symbol R
- added D9: D_TVS, footprint:DO-214AC(SMA), symbol D_TVS
- added SW1: SW_Push, Buttons_Switches_THT:SW_PUSH_6mm_h4.3mm, symbol SW_Push
Connections:
- net GND: now also D9.2 (A2), SW1.1
- net at U5.39 (PWRKEY): now also D9.1 (A1), SW1.2
Changed lines of the file:
@@
-$EndComp
-$Comp
-L R R15
-U 1 1 59DF4296
-P 4675 3600
-F 0 "R15" V 4755 3600 50  0000 C CNN
-F 1 "10k" V 4675 3600 50  0000 C CNN
-F 2 "footprint:R_0603" V 4605 3600 50  0001 C CNN
-F 3 "" H 4675 3600 50  0001 C CNN
-	1    4675 3600
-	0    1    1    0
 $EndComp
 $Comp
@@
 	7625 4900 7525 4900
 Wire Wire Line
-	4950 3600 4825 3600
-Wire Wire Line
-	4525 3600 4375 3600
-Wire Wire Line
-	4375 3600 4375 3675
+	4525 3600 4950 3600
+Wire Wire Line
+	3900 3600 4125 3600
+Wire Wire Line
+	3900 3600 3900 3675
 Wire Wire Line
 	4600 4900 4950 4900
@@
 Text HLabel 2900 2450 0    60   Input ~ 0
 GND
-Text HLabel 4375 3675 3    60   Input ~ 0
+Text HLabel 3900 3675 3    60   Input ~ 0
 GND
 $Comp
@@
 	1    0    0    -1
 $EndComp
+$Comp
+L D_TVS D9
+U 1 1 59DD9C2C
+P 4700 3800
+F 0 "D9" H 4700 3900 50  0000 C CNN
+F 1 "D_TVS" H 4700 3700 50  0000 C CNN
+F 2 "footprint:DO-214AC(SMA)" H 4700 3800 50  0001 C CNN
+F 3 "" H 4700 3800 50  0001 C CNN
+	1    4700 3800
+	0    1    1    0
+$EndComp
+Wire Wire Line
+	4700 3600 4700 3650
+$Comp
+L SW_Push SW1
+U 1 1 59DD9D26
+P 4325 3600
+F 0 "SW1" H 4375 3700 50  0000 L CNN
+F 1 "SW_Push" H 4325 3540 50  0000 C CNN
+F 2 "Buttons_Switches_THT:SW_PUSH_6mm_h4.3mm" H 4325 3800 50  0001 C CNN
+F 3 "" H 4325 3800 50  0001 C CNN
+	1    4325 3600
+	1    0    0    -1
+$EndComp
+Connection ~ 4700 3600
+Text HLabel 4550 4025 0    60   Input ~ 0
+GND
+Wire Wire Line
+	4700 3950 4700 4025
+Wire Wire Line
+	4700 4025 4550 4025
 $EndSCHEMATC

Commit message: Make PCB
Parts:
- J7: footprint (none) -> footprint:MOLEX_47553-2001_SIMCARD
Changed lines of the file:
@@
 $EndComp
 $Comp
-L GND #PWR26
+L GND #PWR026
 U 1 1 59DF42A3
 P 4300 2425
-F 0 "#PWR26" H 4300 2175 50  0001 C CNN
+F 0 "#PWR026" H 4300 2175 50  0001 C CNN
 F 1 "GND" H 4300 2275 50  0000 C CNN
 F 2 "" H 4300 2425 50  0001 C CNN
@@
 F 0 "J7" H 9500 3900 50  0000 R CNN
 F 1 "SIM_Card" H 9550 3800 50  0000 R CNN
-F 2 "" H 9600 3750 50  0000 C CNN
+F 2 "footprint:MOLEX_47553-2001_SIMCARD" H 9600 3750 50  0001 C CNN
 F 3 "" H 9550 3400 50  0000 C CNN
 	1    9600 3400

Commit message: add PCB
Parts:
- added C23: 10uF, footprint:C_0603, symbol C
- added C24: 100nF, footprint:C_0603, symbol C
- D7: footprint footprint:R_0603 -> LEDs:LED_D3.0mm
Connections:
- net 3.3V: now also C23.1, C24.1
- net GND: now also J6.2, C23.2, C24.2; no longer J6.1
- net at C17.1, R14.2: now also J6.1; no longer J6.2
Changed lines of the file:
@@
 LIBS:SIM800C
 LIBS:MCP1727-3302E_SN
+LIBS:MOSFET-N
+LIBS:MOSFET-P
 LIBS:esp32-gateway-hw-cache
 EELAYER 25 0
@@
 F 0 "D7" H 7375 5000 50  0000 C CNN
 F 1 "LED" H 7375 4800 50  0000 C CNN
-F 2 "footprint:R_0603" H 7375 4900 50  0001 C CNN
+F 2 "LEDs:LED_D3.0mm" H 7375 4900 50  0001 C CNN
 F 3 "" H 7375 4900 50  0001 C CNN
 	1    7375 4900
@@
 F 3 "" H 3700 4950 50  0001 C CNN
 	1    3700 4950
-	-1   0    0    1
+	-1   0    0    -1
 $EndComp
 $Comp
@@
 $EndComp
 $Comp
-L GND #PWR26
+L GND #PWR028
 U 1 1 59DF42A3
 P 4300 2425
-F 0 "#PWR26" H 4300 2175 50  0001 C CNN
+F 0 "#PWR028" H 4300 2175 50  0001 C CNN
 F 1 "GND" H 4300 2275 50  0000 C CNN
 F 2 "" H 4300 2425 50  0001 C CNN
@@
 NoConn ~ 6750 4000
 NoConn ~ 6750 3600
-Wire Notes Line
-	12150 1450 12150 1400
-Wire Wire Line
-	6750 3100 9100 3100
-Wire Wire Line
-	7450 3200 9100 3200
-Wire Wire Line
-	7100 3200 6800 3300
-Wire Wire Line
-	6800 3300 6750 3300
-Wire Wire Line
-	7150 3300 7100 3300
-Wire Wire Line
-	7100 3300 6800 3200
-Wire Wire Line
-	6800 3200 6750 3200
-Wire Wire Line
-	7100 3200 7150 3200
-Wire Wire Line
-	7450 3300 9100 3300
-Wire Wire Line
-	4750 3300 4950 3300
-Wire Wire Line
-	7300 3400 9100 3400
-Wire Wire Line
-	7300 3400 7300 4100
-Connection ~ 7650 3100
-Wire Wire Line
-	7650 3450 7650 3100
-Wire Wire Line
-	7300 4100 8550 4100
-Wire Wire Line
-	7650 3750 7650 4225
-Connection ~ 7650 4100
-Wire Wire Line
-	9000 3600 9100 3600
-Wire Wire Line
-	8700 3600 8700 3700
-Wire Wire Line
-	8550 3700 8850 3700
-Wire Wire Line
-	8550 3700 8550 3750
-Wire Wire Line
-	8850 3700 8850 3750
-Connection ~ 8700 3700
-Wire Wire Line
-	8550 4100 8550 4050
-Connection ~ 8350 3100
-Connection ~ 8250 3200
-Wire Wire Line
-	8350 3100 8350 3475
-Wire Wire Line
-	8250 3200 8250 3475
-Wire Wire Line
-	8150 3300 8150 3475
-Connection ~ 8150 3300
-Wire Wire Line
-	8050 3400 8050 3475
-Connection ~ 8050 3400
-Wire Wire Line
-	8150 4075 8150 4100
-Connection ~ 8150 4100
-Wire Wire Line
-	6875 5100 6875 5000
-Wire Wire Line
-	6875 5000 6750 5000
-Wire Wire Line
-	6925 2800 6750 2800
-Wire Wire Line
-	6925 2500 6925 2800
-Wire Wire Line
-	6750 2700 6925 2700
-Connection ~ 6925 2700
-Wire Wire Line
-	4950 4200 4750 4200
-Wire Wire Line
-	4950 4300 4750 4300
-Wire Wire Line
-	6850 4900 6750 4900
-Wire Wire Line
-	7150 4900 7225 4900
-Wire Wire Line
-	7625 5100 7625 4900
-Wire Wire Line
-	7625 4900 7525 4900
-Wire Wire Line
-	4525 3600 4950 3600
-Wire Wire Line
-	3900 3600 4125 3600
-Wire Wire Line
-	3900 3600 3900 3675
-Wire Wire Line
-	4600 4900 4950 4900
-Wire Wire Line
-	4000 4900 4300 4900
-Wire Wire Line
-	4200 4900 4200 4975
-Connection ~ 4200 4900
-Wire Wire Line
-	4725 4975 4725 4900
-Connection ~ 4725 4900
-Wire Wire Line
-	4725 5375 4725 5275
-Wire Wire Line
-	4200 5375 4200 5275
-Wire Wire Line
-	4475 5375 4475 5450
-Connection ~ 4475 5375
-Connection ~ 4200 5375
-Wire Wire Line
-	4000 5000 4025 5000
-Wire Wire Line
-	4025 5000 4025 5375
-Wire Wire Line
-	4025 5375 4725 5375
-Wire Wire Line
-	4525 2800 4950 2800
-Wire Wire Line
-	3800 2900 4950 2900
-Wire Wire Line
-	3400 3000 4950 3000
-Wire Wire Line
-	2900 2450 2950 2450
-Wire Wire Line
-	2950 2200 2950 2725
-Wire Wire Line
-	2950 2725 3050 2725
-Wire Wire Line
-	2950 2200 3050 2200
-Connection ~ 2950 2450
-Wire Wire Line
-	3350 2200 3475 2200
-Wire Wire Line
-	3775 2200 3875 2200
-Wire Wire Line
-	4250 2200 4175 2200
-Wire Wire Line
-	4250 2200 4250 2725
-Wire Wire Line
-	4250 2425 4300 2425
-Wire Wire Line
-	4250 2725 4175 2725
-Connection ~ 4250 2425
-Wire Wire Line
-	3750 2725 3875 2725
-Wire Wire Line
-	3350 2725 3450 2725
-Connection ~ 3800 2725
-Connection ~ 3800 2200
-Wire Wire Line
-	3400 1950 3400 3000
-Connection ~ 3400 2725
-Connection ~ 3400 2200
-Wire Wire Line
-	3800 2000 3800 2900
-Wire Wire Line
-	4625 1525 4625 2700
-Wire Wire Line
-	4525 1525 4525 2800
-Wire Wire Line
-	4425 2000 3800 2000
-Wire Wire Line
-	4425 1525 4425 2000
-Wire Wire Line
-	4325 1525 4325 1950
-Wire Wire Line
-	4325 1950 3400 1950
-Wire Wire Line
-	4625 2700 4950 2700
 Text HLabel 4750 4300 0    60   Input ~ 0
 SIM_RXD
@@
 	0    1    1    0
 $EndComp
-Wire Wire Line
-	4700 3600 4700 3650
 $Comp
 L SW_Push SW1
@@
 	1    0    0    -1
 $EndComp
+Text HLabel 4550 4025 0    60   Input ~ 0
+GND
+Text HLabel 7625 2325 1    60   Input ~ 0
+3.3V
+$Comp
+L C C24
+U 1 1 59E77FAA
+P 7625 2475
+F 0 "C24" H 7650 2575 50  0000 L CNN
+F 1 "100nF" H 7650 2375 50  0000 L CNN
+F 2 "footprint:C_0603" H 7663 2325 50  0001 C CNN
+F 3 "" H 7625 2475 50  0001 C CNN
+	1    7625 2475
+	1    0    0    -1
+$EndComp
+$Comp
+L GND #PWR029
+U 1 1 59E7800F
+P 7625 2625
+F 0 "#PWR029" H 7625 2375 50  0001 C CNN
+F 1 "GND" H 7625 2475 50  0000 C CNN
+F 2 "" H 7625 2625 50  0001 C CNN
+F 3 "" H 7625 2625 50  0001 C CNN
+	1    7625 2625
+	1    0    0    -1
+$EndComp
+Text HLabel 7375 2325 1    60   Input ~ 0
+3.3V
+$Comp
+L C C23
+U 1 1 59E783BD
+P 7375 2475
+F 0 "C23" H 7400 2575 50  0000 L CNN
+F 1 "10uF" H 7400 2375 50  0000 L CNN
+F 2 "footprint:C_0603" H 7413 2325 50  0001 C CNN
+F 3 "" H 7375 2475 50  0001 C CNN
+	1    7375 2475
+	1    0    0    -1
+$EndComp
+$Comp
+L GND #PWR030
+U 1 1 59E783C3
+P 7375 2625
+F 0 "#PWR030" H 7375 2375 50  0001 C CNN
+F 1 "GND" H 7375 2475 50  0000 C CNN
+F 2 "" H 7375 2625 50  0001 C CNN
+F 3 "" H 7375 2625 50  0001 C CNN
+	1    7375 2625
+	1    0    0    -1
+$EndComp
+Wire Notes Line
+	12150 1450 12150 1400
+Wire Wire Line
+	6750 3100 9100 3100
+Wire Wire Line
+	7450 3200 9100 3200
+Wire Wire Line
+	7100 3200 6800 3300
+Wire Wire Line
+	6800 3300 6750 3300
+Wire Wire Line
+	7150 3300 7100 3300
+Wire Wire Line
+	7100 3300 6800 3200
+Wire Wire Line
+	6800 3200 6750 3200
+Wire Wire Line
+	7100 3200 7150 3200
+Wire Wire Line
+	7450 3300 9100 3300
+Wire Wire Line
+	4750 3300 4950 3300
+Wire Wire Line
+	7300 3400 9100 3400
+Wire Wire Line
+	7300 3400 7300 4100
+Connection ~ 7650 3100
+Wire Wire Line
+	7650 3450 7650 3100
+Wire Wire Line
+	7300 4100 8550 4100
+Wire Wire Line
+	7650 3750 7650 4225
+Connection ~ 7650 4100
+Wire Wire Line
+	9000 3600 9100 3600
+Wire Wire Line
+	8700 3600 8700 3700
+Wire Wire Line
+	8550 3700 8850 3700
+Wire Wire Line
+	8550 3700 8550 3750
+Wire Wire Line
+	8850 3700 8850 3750
+Connection ~ 8700 3700
+Wire Wire Line
+	8550 4100 8550 4050
+Connection ~ 8350 3100
+Connection ~ 8250 3200
+Wire Wire Line
+	8350 3100 8350 3475
+Wire Wire Line
+	8250 3200 8250 3475
+Wire Wire Line
+	8150 3300 8150 3475
+Connection ~ 8150 3300
+Wire Wire Line
+	8050 3400 8050 3475
+Connection ~ 8050 3400
+Wire Wire Line
+	8150 4075 8150 4100
+Connection ~ 8150 4100
+Wire Wire Line
+	6875 5100 6875 5000
+Wire Wire Line
+	6875 5000 6750 5000
+Wire Wire Line
+	6925 2800 6750 2800
+Wire Wire Line
+	6925 2500 6925 2800
+Wire Wire Line
+	6750 2700 6925 2700
+Connection ~ 6925 2700
+Wire Wire Line
+	4950 4200 4750 4200
+Wire Wire Line
+	4950 4300 4750 4300
+Wire Wire Line
+	6850 4900 6750 4900
+Wire Wire Line
+	7150 4900 7225 4900
+Wire Wire Line
+	7625 5100 7625 4900
+Wire Wire Line
+	7625 4900 7525 4900
+Wire Wire Line
+	4525 3600 4950 3600
+Wire Wire Line
+	3900 3600 4125 3600
+Wire Wire Line
+	3900 3600 3900 3675
+Wire Wire Line
+	4600 4900 4950 4900
+Wire Wire Line
+	4000 4900 4300 4900
+Wire Wire Line
+	4200 4900 4200 4975
+Connection ~ 4200 4900
+Wire Wire Line
+	4725 4975 4725 4900
+Connection ~ 4725 4900
+Wire Wire Line
+	4725 5375 4725 5275
+Wire Wire Line
+	4200 5375 4200 5275
+Wire Wire Line
+	4475 5375 4475 5450
+Connection ~ 4475 5375
+Connection ~ 4200 5375
+Wire Wire Line
+	4000 5000 4025 5000
+Wire Wire Line
+	4025 5000 4025 5375
+Wire Wire Line
+	4025 5375 4725 5375
+Wire Wire Line
+	4525 2800 4950 2800
+Wire Wire Line
+	3800 2900 4950 2900
+Wire Wire Line
+	3400 3000 4950 3000
+Wire Wire Line
+	2900 2450 2950 2450
+Wire Wire Line
+	2950 2200 2950 2725
+Wire Wire Line
+	2950 2725 3050 2725
+Wire Wire Line
+	2950 2200 3050 2200
+Connection ~ 2950 2450
+Wire Wire Line
+	3350 2200 3475 2200
+Wire Wire Line
+	3775 2200 3875 2200
+Wire Wire Line
+	4250 2200 4175 2200
+Wire Wire Line
+	4250 2200 4250 2725
+Wire Wire Line
+	4250 2425 4300 2425
+Wire Wire Line
+	4250 2725 4175 2725
+Connection ~ 4250 2425
+Wire Wire Line
+	3750 2725 3875 2725
+Wire Wire Line
+	3350 2725 3450 2725
+Connection ~ 3800 2725
+Connection ~ 3800 2200
+Wire Wire Line
+	3400 1950 3400 3000
+Connection ~ 3400 2725
+Connection ~ 3400 2200
+Wire Wire Line
+	3800 2000 3800 2900
+Wire Wire Line
+	4625 1525 4625 2700
+Wire Wire Line
+	4525 1525 4525 2800
+Wire Wire Line
+	4425 2000 3800 2000
+Wire Wire Line
+	4425 1525 4425 2000
+Wire Wire Line
+	4325 1525 4325 1950
+Wire Wire Line
+	4325 1950 3400 1950
+Wire Wire Line
+	4625 2700 4950 2700
+Wire Wire Line
+	4700 3600 4700 3650
 Connection ~ 4700 3600
-Text HLabel 4550 4025 0    60   Input ~ 0
-GND
 Wire Wire Line
 	4700 3950 4700 4025
